Commit message: minor changes for readability

File: ros2/description/urdf/colors.xacro (robot description, xacro)
@@ -1,3 +1,3 @@
-<?xml version="1.0"?>
+<?xml version="1.0" encoding="utf-8"?>
 <robot xmlns:xacro="http://www.ros.org/wiki/xacro">
   <!-- Misc. colors for making different parts easier to identify -->

File: ros2/description/urdf/sensors.xacro (robot description, xacro)
@@ -4,8 +4,8 @@
   <joint name="laser_joint" type="fixed">
     <parent link="chassis_link" />
-    <child link="laser_frame" />
+    <child link="laser_link" />
     <origin xyz="0 0 0.1" rpy="0 0 0" />
   </joint>
-  <link name="laser_frame">
+  <link name="laser_link">
     <visual>
       <geometry>
@@ -37,9 +37,9 @@
     </visual>
   </link>
-  <joint name="camera_optical_joint" type="fixed">
+  <!-- <joint name="camera_optical_joint" type="fixed">
     <parent link="camera_link" />
     <child link="camera_link_optical" />
     <origin xyz="0 0 0" rpy="${-pi/2} 0 ${-pi/2}" />
   </joint>
-  <link name="camera_link_optical"></link>
+  <link name="camera_link_optical"></link> -->
 </robot>
